Commit message: Configure the exemplo 9 to run in gazebo fortress

File: example_9/description/gazebo/rrbot.gazebo.xacro (robot description, xacro)
@@ -5,11 +5,21 @@
 -->
 <robot xmlns:xacro="http://ros.org/wiki/xacro">
-  <xacro:macro name="rrbot_gazebo" params="prefix">
-    <!-- ros_control plugin -->
-    <gazebo>
-      <plugin filename="libgazebo_ros2_control.so" name="gazebo_ros2_control">
-        <parameters>$(find ros2_control_demo_example_9)/config/rrbot_controllers.yaml</parameters>
-      </plugin>
-    </gazebo>
+  <xacro:macro name="rrbot_gazebo" params="prefix gazebo_fortress:=^|true">
+    <xacro:if value="${gazebo_fortress}">
+      <!-- Gazebo Fortress ros_control plugin -->
+      <gazebo>
+        <plugin filename="ign_ros2_control-system" name="ign_ros2_control::IgnitionROS2ControlPlugin">
+          <parameters>$(find ros2_control_demo_example_9)/config/rrbot_controllers.yaml</parameters>
+        </plugin>
+      </gazebo>
+    </xacro:if>
+    <xacro:unless value="${gazebo_fortress}">
+      <!-- Gazebo Classic ros_control plugin -->
+      <gazebo>
+        <plugin filename="libgazebo_ros2_control.so" name="gazebo_ros2_control">
+          <parameters>$(find ros2_control_demo_example_9)/config/rrbot_controllers.yaml</parameters>
+        </plugin>
+      </gazebo>
+    </xacro:unless>
     <!-- Link1 -->
     <gazebo reference="${prefix}base_link">

File: example_9/description/ros2_control/rrbot.ros2_control.xacro (robot description, xacro)
@@ -1,11 +1,16 @@
 <?xml version="1.0"?>
 <robot xmlns:xacro="http://www.ros.org/wiki/xacro">
-  <xacro:macro name="rrbot_ros2_control" params="name prefix use_gazebo_classic:=^|false">
+  <xacro:macro name="rrbot_ros2_control" params="name prefix use_gazebo:=^|false gazebo_fortress:=^|true">
     <ros2_control name="${name}" type="system">
       <hardware>
-        <xacro:if value="${use_gazebo_classic}">
-          <plugin>gazebo_ros2_control/GazeboSystem</plugin>
+        <xacro:if value="${use_gazebo}">
+          <xacro:if value="${gazebo_fortress}">
+            <plugin>ign_ros2_control/IgnitionSystem</plugin>
+          </xacro:if>
+          <xacro:unless value="${gazebo_fortress}">
+            <plugin>gazebo_ros2_control/GazeboSystem</plugin>
+          </xacro:unless>
         </xacro:if>
-        <xacro:unless value="${use_gazebo_classic}">
+        <xacro:unless value="${use_gazebo}">
           <plugin>ros2_control_demo_example_9/RRBotSystemPositionOnlyHardware</plugin>
           <param name="example_param_hw_start_duration_sec">0</param>

File: example_9/description/urdf/rrbot.urdf.xacro (robot description, xacro)
@@ -7,5 +7,6 @@
 <robot xmlns:xacro="http://www.ros.org/wiki/xacro" name="2dof_robot">
   <xacro:arg name="prefix" default="" />
-  <xacro:arg name="use_gazebo_classic" default="false" />
+  <xacro:arg name="use_gazebo" default="false" />
+  <xacro:arg name="gazebo_fortress" default="true" />
   <!-- Import RRBot macro -->
   <xacro:include filename="$(find ros2_control_demo_description)/rrbot/urdf/rrbot_description.urdf.xacro" />
@@ -20,9 +21,9 @@
   </xacro:rrbot>
   <xacro:rrbot_ros2_control
-    name="RRBot" prefix="$(arg prefix)" use_gazebo_classic="$(arg use_gazebo_classic)"/>
-  <xacro:if value="$(arg use_gazebo_classic)">
+    name="RRBot" prefix="$(arg prefix)" use_gazebo="$(arg use_gazebo)" gazebo_fortress="$(arg gazebo_fortress)"/>
+  <xacro:if value="$(arg use_gazebo)">
     <!-- Import Gazebo Classic definitions + plugin -->
     <xacro:include filename="$(find ros2_control_demo_example_9)/gazebo/rrbot.gazebo.xacro" />
-    <xacro:rrbot_gazebo prefix="$(arg prefix)"/>
+    <xacro:rrbot_gazebo prefix="$(arg prefix)" gazebo_fortress="$(arg gazebo_fortress)"/>
   </xacro:if>
 </robot>
